File: ntsc_syncgen/ntsc_syncgen.kicad_sch (KiCad schematic)
At the start: 12 parts, among them Q1 PN2222A, U1 74HC4040D, U2 74HC4040D, U3 74HC7014, U4 74HC74D, Y1 Crystal

Commit message: example circuit
Parts:
- added U5: 74HC00, Package_DIP:DIP-14_W7.62mm_SMDSocket_SmallPads, symbol 74xx:74HC00
- added U6, U7, U8: 4081, Package_DIP:DIP-14_W7.62mm_SMDSocket_SmallPads, symbol 4xxx:4081
- added U9: 4001, Package_DIP:DIP-14_W8.89mm_SMDSocket_LongPads, symbol 4xxx:4001
Connections:
- net 14.318mhz_CLK0: now also U3.4, U4.3 (1CP)
- net 7.1mhz_CLK1: now reaches U4.5 (1Q)
- net 7.1mhz_CLK1: now also U2.10 (CP*)
- net 128H: now reaches U2.12 (Q8)
- net 64H: now reaches U2.13 (Q7)
- net 256H: now reaches U2.14 (Q9)
- net 512H: now reaches U2.15 (Q10)
- net 16H: now reaches U2.2 (Q5)
- net 8H: now reaches U2.3 (Q4)
- net 32H: now reaches U2.4 (Q6)
- net 4H: now reaches U2.5 (Q3)
- net 2H: now reaches U2.6 (Q2)
- net 1H: now reaches U2.7 (Q1)
- net H_RESET: now reaches U1.10 (CP*)
- net 128V: now reaches U1.12 (Q8)
- net 64V: now reaches U1.13 (Q7)
- net 256V: now reaches U1.14 (Q9)
- net 512V: now reaches U1.15 (Q10)
- net 16V: now reaches U1.2 (Q5)
- net 8V: now reaches U1.3 (Q4)
- net 32V: now reaches U1.4 (Q6)
- net 4V: now reaches U1.5 (Q3)
- net 2V: now reaches U1.6 (Q2)
- net 1V: now reaches U1.7 (Q1)
- no-connect marks 0 -> 2
Other:
- moved on the sheet: U1, U2, U4

Commit message: more work
Parts:
- removed U4: 74HC74D, footprints:SOT109-1_NXP, symbol 74hc74d:74HC74D
- removed U8: 4081, Package_DIP:DIP-14_W7.62mm_SMDSocket_SmallPads, symbol 4xxx:4081
- added U10: 74HC74, Library:SOIC127P600X175-14N, symbol 74xx:74HC74
- U5, U6, U7: footprint Package_DIP:DIP-14_W7.62mm_SMDSocket_SmallPads -> Package_SO:SOIC-14_3.9x8.7mm_P1.27mm
- U9: footprint Package_DIP:DIP-14_W8.89mm_SMDSocket_LongPads -> Package_SO:SOIC-14_3.9x8.7mm_P1.27mm
Connections:
- net 128H: now also U7.6
- net 128V: now also U1.13 (Q7); no longer U1.12 (Q8)
- net 14.318mhz_CLK0: now also U2.10 (CP*)
- net 16H: now also U5.1
- net 16V: now also U1.3 (Q4), U9.6; no longer U1.2 (Q5)
- net 1V: now also U1.9 (Q0), U6.6; no longer U1.7 (Q1)
- net 256H: now also U7.13
- net 256V: now also U1.12 (Q8), U6.1; no longer U1.14 (Q9)
- net 2H: now also U7.1
- net 2V: now also U1.7 (Q1); no longer U1.6 (Q2)
- net 32H: now also U5.13
- net 32V: now also U1.2 (Q5); no longer U1.4 (Q6)
- net 4H: now also U7.2
- net 4V: now also U1.6 (Q2), U6.2, U9.13; no longer U1.5 (Q3)
- net 512V: now also U1.14 (Q9); no longer U1.15 (Q10)
- net 64H: now also U5.2, U7.5
- net 64V: now also U1.4 (Q6); no longer U1.13 (Q7)
- net 7.1mhz_CLK1: now also U2.9 (Q0), U10.3 (C); no longer U2.10 (CP*)
- net 8V: now also U1.5 (Q3), U3.9; no longer U1.3 (Q4)
- net GND: now also U5.7 (GND), U6.7 (VSS), U7.7 (VSS), U9.7 (VSS), U10.7 (GND)
- net H_RESET: now also U2.11 (MR), U10.6 (~{Q})
- net VCC: now also U5.14 (VCC), U6.14 (VDD), U7.14 (VDD), U9.14 (VDD), U10.14 (VCC)
- net V_RESET: now reaches U9.1
- net VBLANK: now reaches U9.2
- net VBLANK: now also U9.4, U9.8
- net _VBLANK: now reaches U9.3
- net _VBLANK: now also U9.5
- net at U9.10: now also U9.12
- net at U9.9: now also U3.8
- net at U5.10: now also U5.12, U5.6
- net H_BLANK: now reaches U5.8
- net H_BLANK: now also U5.4
- net at U5.9: now also U3.6
- net at U7.4: now also U7.12
- net at U6.3: now also U6.5
- net _H_RESET: now reaches U5.5
- net _H_RESET: now also U10.5 (Q)
- net at U7.3: now also U7.8
- net at U7.10: now also U10.2 (D)
- net at U7.9: now also U7.11
- net _H_SYNC: now reaches U5.11
- net _VSYNC: now reaches U9.11
- net at U5.3: now also U3.5
- net at U6.4: now also U10.12 (D)
- new net HRESET: U10.11 (C)
- new net VRESET: U10.8 (~{Q})
- no-connect marks 2 -> 3
Other:
- note added: "1H - Q1 is 3.5795mhz colorburst period of 279.36nS"
- note added: "H_Reset is the clock source for Vertical counter activates once its time to draw a new horizontal line this increments the vertical counter +1"
- note added: "crystal is 14.318mhz circuit timing is /2 so 1H is actually /4 or Q1 and clock source is /2 or Q0"
- note added: "spare parts bin"
- note added: "these capacitors might not be needed"
- moved on the sheet: U3C, U3D, U3E, U3F, U3G, U5A, U5B, U5C, U5D, U5E, U6A, U6B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
